File: Hardware/GRBLShieldv2.brd (EAGLE design)
At the start: 150 x 80 mm, 169 parts, among them J1 AVR ISP, Q1 16MHZ, Q2 100A/100V, U1 ATMEGA328, U2 CY7C65213, U3 74LVC1G04, U4 LM25011, U5 DRV8811, U6 74HC7014D, U7 74AHC1G08, U8 DRV8811, U9 DRV8811

Commit message: schematic cleanup
Parts:
- removed JP7: Power, SparkFun-Connectors:SCREWTERMINAL-5MM-2
- added VIN: 3.5mm, SparkFun-Connectors:SCREWTERMINAL-3.5MM-2_LOCK
- JP1, JP3, JP4, JP8, JP9: value M023.5MM -> 3.5mm; device SparkFun-Connectors:SCREWTERMINAL-3.5MM-2 -> SparkFun-Connectors:SCREWTERMINAL-3.5MM-2_LOCK
- JP15: value Fan -> 3.5mm; device SparkFun-Connectors:SCREWTERMINAL-5MM-2 -> SparkFun-Connectors:SCREWTERMINAL-3.5MM-2_LOCK
- POT1, POT2, POT3: value (none) -> 2K_LINEAR_POT_SMD; device adafruit:TC33X -> SparkFun-Resistors:TC33X
- R1, R17, R26: value 680 -> 240
- R16, R25, R37: value 2.4K -> 1K
- R6: device SparkFun:0603-RES -> SparkFun-Resistors:0603-RES
- X-A, Y-A, Z-A: value A -> 3.5mm
- X-B, Y-B, Z-B: value B -> 3.5mm
- renumbered JP10 to X-B, JP11 to Y-A, JP12 to Y-B, JP13 to Z-A, JP14 to Z-B, JP2 to X-A
Connections:
- net N$17: now also VIN.1; no longer JP7.1
- net VIN: now also VIN.2; no longer JP7.2
Routing:
- net VCC: track 47.0 -> 45.6 mm
- net VIN: track 84.5 -> 84.0 mm

Commit message: cleanup
Parts:
- removed 12V: UA78M12, texas:TO-252
- removed D3: MBRA140, SparkFun-DiscreteSemi:SMA-DIODE
- added POWER: BLUE, SparkFun-LED:LED-1206
- added PROTECT: RED, SparkFun-LED:LED-1206
- added R56: 10K, SparkFun-Resistors:0603-RES
- added SJ1: Limit Pull Direction, SparkFun-Passives:PAD-JUMPER-3-2OF3_NC_BY_TRACE_YES_SILK_LARGE
- added U10: (no value), SparkFun-PowerIC:TO-252
- D10: value Y_Lim (Yellow) -> YELLOW
- D11: value PROBE (Blue) -> BLUE
- D12: value Z_STEP (Green) -> GREEN
- D13: value Z_DIR (Red) -> RED
- D14: value Z_Lim (Yellow) -> YELLOW
- D15: value STEP_EN (Green) -> GREEN
- D16: value PROTECT -> MBRA140; device SparkFun-LED:LED-1206 -> SparkFun-DiscreteSemi:SMA-DIODE
- D4: value X_STEP (Green) -> GREEN
- D5: value X_DIR (Red) -> RED
- D6: value X_Lim (Yellow) -> YELLOW
- D7: value ESTOP (Red) -> RED
- D8: value Y_STEP (Green) -> GREEN
- D9: value Y_DIR (Red) -> RED
- R12, R13, R14, R15, R21, R22, R23, R24, R4, R5, R7, R8: device SparkFun-Resistors:0603-RES -> SparkFun-Resistors:0603
- R53: value (none) -> 9.76K
- R54: value (none) -> 50.0m
- R55: value (none) -> 348K
- S1, S2, S3: value CHS-02A -> 2-POS-DIP; device switch-copal:CHS-02A -> SparkFun-Electromechanical:CHS-02A
- moved D16 20.1 mm to (139.0, 34.5), turned to 90 degrees
Connections:
- removed net N$1: U2.5
- removed net N$4: U2.1
- new net N$62: POWER.A, R56.2
- new net N$95: R27.1, R28.1, R38.1, SJ1.2
- net 5V: now also D16.C, SJ1.3; no longer D3.C, JP16.4, R27.1, R28.1, R38.1
- net ESTOP: now also JP16.4
- net GND: now also POWER.C, SJ1.1, U10.3; no longer 12V.3
- net N$17: now also PROTECT.A; no longer D16.A
- net N$41: now also PROTECT.C; no longer D16.C
- net N$51: now also D16.A; no longer D3.A
- net RXI: now also U2.1
- net TXO: now also U2.5
- net VCC: now also U10.2; no longer 12V.2
- net VIN: now also R56.1, U10.1; no longer 12V.1
Routing:
- net TXO: track 39.3 -> 91.5 mm, vias 0 -> 1
- net RXI: track 43.0 -> 94.3 mm, vias 0 -> 1
- net N$95: track 0.00 -> 35.6 mm, vias 0 -> 4
- net 5V: track 546.4 -> 521.0 mm, vias 35 -> 33
- net ESTOP: track 90.1 -> 97.2 mm
- net VIN: track 84.0 -> 87.5 mm
- net N$62: track 0.00 -> 3.04 mm
Other:
- board text added: "E-STOP"
- board text added: "Limit"
- board text added: "POWER"
- board text added: "Step En"
- board text added: "Switch Pull +5v-UP GND-DOWN"
