File: Hardware/GRBLShieldv2.sch (EAGLE design)
At the start: 168 parts, among them J1 AVR ISP, Q1 16MHZ, Q2 100A/100V, U1 ATMEGA328, U2 CY7C65213, U3 74LVC1G04, U4 LM25011, U5 DRV8811, U6 74HC7014D, U7 74AHC1G08, U8 DRV8811, U9 DRV8811

Commit message: schematic cleanup
Parts:
- removed JP7: Power, SparkFun-Connectors:M025MM
- added VIN: 3.5mm, SparkFun-Connectors:M023.5MM_LOCK
- FRAME2: DESIGNER (none) -> Casey Kuhns; VERSION (none) -> v02
- JP1, JP3, JP4, JP8, JP9: value M023.5MM -> 3.5mm; device SparkFun-Connectors:M023.5MM -> SparkFun-Connectors:M023.5MM_LOCK
- JP15: value Fan -> 3.5mm; device SparkFun-Connectors:M025MM -> SparkFun-Connectors:M023.5MM_LOCK
- POT1, POT2, POT3: value (none) -> 2K_LINEAR_POT_SMD; device adafruit:TRIMPOTTC33X -> SparkFun-Resistors:2K_LINEAR_POT_SMD
- R1, R17, R26: value 680 -> 240; device SparkFun-Resistors:RESISTOR0603 -> SparkFun-Resistors:240OHM1/10W1%(0603)
- R16, R25, R37: value 2.4K -> 1K; device SparkFun-Resistors:RESISTOR0603 -> SparkFun-Resistors:1KOHM-1/10W-1%(0603)
- R6: device SparkFun:RESISTOR0603-RES -> SparkFun-Resistors:10KOHM-1/10W-1%(0603)0603
- X-A, Y-A, Z-A: value A -> 3.5mm
- X-B, Y-B, Z-B: value B -> 3.5mm
- renumbered JP10 to X-B, JP11 to Y-A, JP12 to Y-B, JP13 to Z-A, JP14 to Z-B, JP2 to X-A
Connections:
- net N$17: now also VIN.1; no longer JP7.1
- net VIN: now also VIN.2; no longer JP7.2
Other:
- note added: "Control Logic"
- note added: "Expansion Headers"
- note added: "Power Management"
- note added: "Status LED's"
- note added: "USB->Serial"
- moved on the sheet: 12V, C2, C39, C4, C40, C41, C42, C5, C50, C51, C52, C53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

Commit message: cleanup
Parts:
- removed 12V: UA78M12, texas:UA78M12
- removed D3: MBRA140, SparkFun-DiscreteSemi:DIODE-SCHOTTKY-MBRA140
- added POWER: BLUE, SparkFun-LED:LED-BLUE1206
- added PROTECT: RED, SparkFun-LED:LED-REDLILYPAD
- added R56: 10K, SparkFun-Resistors:10KOHM-1/10W-1%(0603)0603
- added SJ1: Limit Pull Direction, SparkFun-Passives:JUMPER-PAD-3-2OF3_NC_BY_TRACE_LARGE
- added U10: (no value), SparkFun-PowerIC:V_REG_78XX7812
- D10: value Y_Lim (Yellow) -> YELLOW
- D11: value PROBE (Blue) -> BLUE
- D12: value Z_STEP (Green) -> GREEN
- D13: value Z_DIR (Red) -> RED
- D14: value Z_Lim (Yellow) -> YELLOW
- D15: value STEP_EN (Green) -> GREEN
- D16: value PROTECT -> MBRA140; device SparkFun-LED:LED-REDLILYPAD -> SparkFun-DiscreteSemi:DIODE-SCHOTTKY-MBRA140
- D17: device SparkFun-DiscreteSemi:MBRA140 -> SparkFun-DiscreteSemi:DIODE-SCHOTTKY-MBRA140
- D4: value X_STEP (Green) -> GREEN
- D5: value X_DIR (Red) -> RED
- D6: value X_Lim (Yellow) -> YELLOW
- D7: value ESTOP (Red) -> RED
- D8: value Y_STEP (Green) -> GREEN
- D9: value Y_DIR (Red) -> RED
- R12, R13, R21, R22, R4, R5: device SparkFun-Resistors:RESISTOR0603 -> SparkFun-Resistors:39KOHM-1/10W-1%(0603)
- R14, R15, R23, R24, R7, R8: device SparkFun-Resistors:RESISTOR0603 -> SparkFun-Resistors:5.6KOHM-1/10W-1%(0603)
- R27, R28, R29, R35, R38, R51, R52: device SparkFun-Resistors:10KOHM1/10W1%(0603)0603 -> SparkFun-Resistors:10KOHM-1/10W-1%(0603)0603
- R53: value (none) -> 9.76K
- R54: value (none) -> 50.0m
- R55: value (none) -> 348K
- S1, S2, S3: value CHS-02A -> 2-POS-DIP; device switch-copal:CHS-02A -> SparkFun-Electromechanical:2-POS-DIP
Connections:
- removed net N$1: U2.RXD
- removed net N$4: U2.TXD
- new net N$62: POWER.A, R56.2
- new net N$95: R27.1, R28.1, R38.1, SJ1.2
- net 5V: now also D16.C, S1.P$3, S1.P$4, S2.P$3, S2.P$4, S3.P$3, S3.P$4, SJ1.3; no longer D3.C, JP16.4, R27.1, R28.1, R38.1, S1.3, S1.4, S2.3, S2.4, S3.3, S3.4
- net ESTOP: now also JP16.4
- net GND: now also POWER.C, SJ1.1, U10.GND; no longer 12V.GND
- net N$15: now also S2.P$2; no longer S2.2
- net N$17: now also PROTECT.A; no longer D16.A
- net N$23: now also S2.P$1; no longer S2.1
- net N$34: now also S1.P$2; no longer S1.2
- net N$35: now also S1.P$1; no longer S1.1
- net N$41: now also PROTECT.C; no longer D16.C
- net N$51: now also D16.A; no longer D3.A
- net N$76: now also S3.P$2; no longer S3.2
- net N$77: now also S3.P$1; no longer S3.1
- net RXI: now also U2.TXD
- net TXO: now also U2.RXD
- net VCC: now also U10.OUT; no longer 12V.OUT
- net VIN: now also R56.1, U10.IN; no longer 12V.IN
Other:
- moved on the sheet: C4
