File: Hardware/Stepoko.sch (EAGLE design)
At the start: 171 parts, among them J1 AVR ISP, Q1 16MHZ, Q2 100A/100V, U1 ATMEGA328, U2 CY7C65213, U3 74LVC1G04, U4 LM25011, U5 DRV8811, U6 74HC7014D, U7 74AHC1G08, U8 DRV8811, U9 DRV8811

Commit message: revision changes from review
Parts:
- added C43: 1000pF, SparkFun-Capacitors:1NF/1000PF-50V-10%(0603)
Connections:
- new net N$1: R54.1, U4.CSG
- net GND: no longer R54.1
Other:
- moved on the sheet: D16, R54
Changed lines of the file:
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@@
 <?xml version="1.0" encoding="utf-8"?>
 <!DOCTYPE eagle SYSTEM "eagle.dtd">
-<eagle version="6.5.0">
+<eagle version="6.6.0">
 <drawing>
 <settings>
@@
 <part name="R53" library="SparkFun-Passives" deviceset="RESISTOR" device="0603-RES" value="9.76K"/>
 <part name="R54" library="SparkFun-Passives" deviceset="RESISTOR" device="0603-RES" value="50.0m"/>
-<part name="GND2" library="SparkFun" deviceset="GND" device=""/>
 <part name="R55" library="SparkFun-Passives" deviceset="RESISTOR" device="0603-RES" value="348K"/>
 <part name="SUPPLY4" library="SparkFun-Aesthetics" deviceset="5V" device=""/>
@@
 <part name="GND67" library="SparkFun" deviceset="GND" device=""/>
 <part name="SUPPLY49" library="SparkFun-Aesthetics" deviceset="5V" device=""/>
+<part name="C43" library="SparkFun-Capacitors" deviceset="1NF/1000PF-50V-10%(0603)" device="" value="1000pF"/>
 </parts>
 <sheets>
@@
 from Board</text>
 <wire x1="55.88" y1="264.16" x2="55.88" y2="248.92" width="0.1524" layer="97" style="shortdash"/>
-<wire x1="55.88" y1="248.92" x2="88.9" y2="248.92" width="0.1524" layer="97" style="shortdash"/>
-<wire x1="88.9" y1="248.92" x2="88.9" y2="264.16" width="0.1524" layer="97" style="shortdash"/>
-<wire x1="88.9" y1="264.16" x2="55.88" y2="264.16" width="0.1524" layer="97" style="shortdash"/>
+<wire x1="55.88" y1="248.92" x2="91.44" y2="248.92" width="0.1524" layer="97" style="shortdash"/>
+<wire x1="91.44" y1="248.92" x2="91.44" y2="264.16" width="0.1524" layer="97" style="shortdash"/>
+<wire x1="91.44" y1="264.16" x2="55.88" y2="264.16" width="0.1524" layer="97" style="shortdash"/>
 <text x="15.24" y="43.18" size="2.54" layer="94" font="vector" ratio="15" align="bottom-center">+</text>
 <text x="15.24" y="38.1" size="2.54" layer="94" font="vector" ratio="15" align="bottom-center">-</text>
@@
 <instance part="P+20" gate="G$1" x="33.02" y="228.6" rot="MR0"/>
 <instance part="F1" gate="G$1" x="63.5" y="254"/>
-<instance part="SUPPLY1" gate="G$1" x="83.82" y="256.54"/>
+<instance part="SUPPLY1" gate="G$1" x="86.36" y="256.54"/>
 <instance part="SUPPLY10" gate="G$1" x="91.44" y="243.84"/>
 <instance part="SUPPLY11" gate="G$1" x="101.6" y="243.84"/>
@@
 <instance part="D17" gate="G$1" x="187.96" y="58.42" rot="R90"/>
 <instance part="R53" gate="G$1" x="213.36" y="55.88" rot="R90"/>
-<instance part="R54" gate="G$1" x="187.96" y="35.56" rot="R90"/>
-<instance part="GND2" gate="1" x="187.96" y="27.94" rot="MR0"/>
+<instance part="R54" gate="G$1" x="180.34" y="48.26"/>
 <instance part="R55" gate="G$1" x="137.16" y="60.96" rot="MR90"/>
 <instance part="SUPPLY4" gate="G$1" x="236.22" y="66.04"/>
@@
 <instance part="R56" gate="G$1" x="76.2" y="60.96" rot="MR270"/>
 <instance part="GND66" gate="1" x="76.2" y="40.64" rot="MR0"/>
-<instance part="D16" gate="G$1" x="73.66" y="254"/>
+<instance part="D16" gate="G$1" x="76.2" y="254"/>
 <instance part="SJ1" gate="G$1" x="403.86" y="256.54" rot="MR90"/>
 <instance part="GND67" gate="1" x="411.48" y="248.92" rot="MR0"/>
@@
 </segment>
 <segment>
-<pinref part="R54" gate="G$1" pin="1"/>
-<pinref part="GND2" gate="1" pin="GND"/>
-</segment>
-<segment>
 <pinref part="C39" gate="G$1" pin="2"/>
 <pinref part="GND32" gate="1" pin="GND"/>
@@
 <net name="5V" class="0">
 <segment>
-<wire x1="76.2" y1="254" x2="83.82" y2="254" width="0.1524" layer="91"/>
-<wire x1="83.82" y1="254" x2="83.82" y2="256.54" width="0.1524" layer="91"/>
+<wire x1="78.74" y1="254" x2="86.36" y2="254" width="0.1524" layer="91"/>
+<wire x1="86.36" y1="254" x2="86.36" y2="256.54" width="0.1524" layer="91"/>
 <pinref part="SUPPLY1" gate="G$1" pin="5V"/>
 <pinref part="D16" gate="G$1" pin="C"/>
@@
 <wire x1="187.96" y1="53.34" x2="187.96" y2="55.88" width="0.1524" layer="91"/>
 <pinref part="R54" gate="G$1" pin="2"/>
-<wire x1="187.96" y1="40.64" x2="187.96" y2="53.34" width="0.1524" layer="91"/>
+<wire x1="185.42" y1="48.26" x2="187.96" y2="48.26" width="0.1524" layer="91"/>
+<wire x1="187.96" y1="48.26" x2="187.96" y2="53.34" width="0.1524" layer="91"/>
 <junction x="187.96" y="53.34"/>
 </segment>
@@
 <pinref part="F1" gate="G$1" pin="2"/>
 <pinref part="D16" gate="G$1" pin="A"/>
+<wire x1="73.66" y1="254" x2="71.12" y2="254" width="0.1524" layer="91"/>
 </segment>
 </net>
@@
 <wire x1="403.86" y1="251.46" x2="403.86" y2="248.92" width="0.1524" layer="91"/>
 <junction x="403.86" y="248.92"/>
+</segment>
+</net>
+<net name="N$1" class="0">
+<segment>
+<pinref part="R54" gate="G$1" pin="1"/>
+<pinref part="U4" gate="G$1" pin="CSG"/>
+<wire x1="175.26" y1="48.26" x2="170.18" y2="48.26" width="0.1524" layer="91"/>
 </segment>
 </net>
@@
 <instance part="SUPPLY41" gate="G$1" x="307.34" y="132.08"/>
 <instance part="SUPPLY42" gate="G$1" x="350.52" y="200.66"/>
+<instance part="C43" gate="G$1" x="17.78" y="177.8" smashed="yes">
+<attribute name="NAME" x="19.304" y="183.261" size="1.27" layer="95"/>
+<attribute name="VALUE" x="19.304" y="180.721" size="1.27" layer="96"/>
+</instance>
 </instances>
 <busses>

Commit message: made changes from design review
Parts:
- removed SJ1: Limit Pull Direction, SparkFun-Passives:JUMPER-PAD-3-2OF3_NC_BY_TRACE_LARGE
- added C45, C46: 0.1uF, SparkFun-Capacitors:0.1UF-25V(+80/-20%)(0603)
- added S5: DPDT, SparkFun-Electromechanical:SWITCH-DPDTAYZ0202
- C43: value 1000pF -> 0.1uF; device SparkFun-Capacitors:1NF/1000PF-50V-10%(0603) -> SparkFun-Capacitors:0.1UF-25V(+80/-20%)(0603)
- S1, S2, S3: value 2-POS-DIP -> 2-POS-DIPCTS-THRU-HOLE; device SparkFun-Electromechanical:2-POS-DIP -> SparkFun-Electromechanical:2-POS-DIPCTS-THRU-HOLE
Connections:
- new net N$4: JP1.1, JP3.1, JP4.1, S5.5
- net 5V: now also S5.1, S5.6; no longer R40.2, SJ1.3
- net ESTOP: now also R40.2; no longer D7.C
- net GND: now also C43.2, C45.2, C46.2, D7.C, S5.3, S5.4; no longer JP1.1, JP3.1, JP4.1, SJ1.1
- net N$95: now also S5.2; no longer SJ1.2
- net VIN: now also C43.1, C45.1, C46.1
Other:
- moved on the sheet: C1, C10, C11, C12, C13, C14, C15, C24, C26, C27, C28, C29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

Commit message: added prod-ids
Parts:
- C15, C32, C36: device SparkFun:CAP0603-CAP -> SparkFun-Capacitors:0.18UF-10V(+-10%)(0603)
- R53: device SparkFun-Passives:RESISTOR0603-RES -> SparkFun-Resistors:9.76KOHM-1/10W-1%(0603)
- R54: device SparkFun-Passives:RESISTOR0603-RES -> SparkFun-Resistors:0.05OHM-1/5W-1%(0603)
- R55: device SparkFun-Passives:RESISTOR0603-RES -> SparkFun-Resistors:348KOHM-1/10W-1%(0603)
Changed lines of the file:
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@@
 <part name="GND11" library="SparkFun" deviceset="GND" device=""/>
 <part name="C23" library="SparkFun-Capacitors" deviceset="47UF-50V-20%(ELECT)" device="" value="47uF"/>
-<part name="C32" library="SparkFun" deviceset="CAP" device="0603-CAP" value="0.18uF"/>
+<part name="C32" library="SparkFun-Capacitors" deviceset="0.18UF-10V(+-10%)(0603)" device="" value="0.18uF"/>
 <part name="GND6" library="SparkFun" deviceset="GND" device=""/>
 <part name="P+18" library="SparkFun" deviceset="VCC" device="" value="12V"/>
@@
 <part name="GND16" library="SparkFun" deviceset="GND" device=""/>
 <part name="C14" library="SparkFun-Capacitors" deviceset="47UF-50V-20%(ELECT)" device="" value="47uF"/>
-<part name="C15" library="SparkFun" deviceset="CAP" device="0603-CAP" value="0.18uF"/>
+<part name="C15" library="SparkFun-Capacitors" deviceset="0.18UF-10V(+-10%)(0603)" device="" value="0.18uF"/>
 <part name="R16" library="SparkFun-Resistors" deviceset="1KOHM-1/10W-1%(0603)" device="" value="1K"/>
 <part name="GND18" library="SparkFun" deviceset="GND" device=""/>
@@
 <part name="GND30" library="SparkFun" deviceset="GND" device=""/>
 <part name="C35" library="SparkFun-Capacitors" deviceset="47UF-50V-20%(ELECT)" device="" value="47uF"/>
-<part name="C36" library="SparkFun" deviceset="CAP" device="0603-CAP" value="0.18uF"/>
+<part name="C36" library="SparkFun-Capacitors" deviceset="0.18UF-10V(+-10%)(0603)" device="" value="0.18uF"/>
 <part name="R25" library="SparkFun-Resistors" deviceset="1KOHM-1/10W-1%(0603)" device="" value="1K"/>
 <part name="GND31" library="SparkFun" deviceset="GND" device=""/>
@@
 <part name="SUPPLY43" library="SparkFun-Aesthetics" deviceset="5V" device=""/>
 <part name="D17" library="SparkFun-DiscreteSemi" deviceset="DIODE-SCHOTTKY" device="-MBRA140" value="MBRA140"/>
-<part name="R53" library="SparkFun-Passives" deviceset="RESISTOR" device="0603-RES" value="9.76K"/>
-<part name="R54" library="SparkFun-Passives" deviceset="RESISTOR" device="0603-RES" value="50.0m"/>
-<part name="R55" library="SparkFun-Passives" deviceset="RESISTOR" device="0603-RES" value="348K"/>
+<part name="R53" library="SparkFun-Resistors" deviceset="9.76KOHM-1/10W-1%(0603)" device="" value="9.76K"/>
+<part name="R54" library="SparkFun-Resistors" deviceset="0.05OHM-1/5W-1%(0603)" device="" value="50.0m"/>
+<part name="R55" library="SparkFun-Resistors" deviceset="348KOHM-1/10W-1%(0603)" device="" value="348K"/>
 <part name="SUPPLY4" library="SparkFun-Aesthetics" deviceset="5V" device=""/>
 <part name="L1" library="SparkFun-Passives" deviceset="INDUCTOR" device="SDR13-7-270ML" value="27uH"/>
