File: Hardware/SparkFun_Stepoko.sch (EAGLE design)
At the start: 174 parts, among them J1 AVR ISP, Q1 16MHZ, Q2 100A/100V, U1 ATMEGA328, U2 CY7C65213, U3 74LVC1G04, U4 LM25011, U5 DRV8811, U6 74HC7014D, U7 74AHC1G08, U8 DRV8811, U9 DRV8811

Commit message: made changes from design review
Connections:
- net GND: now also U6.6A
Changed lines of the file:
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@@
 <?xml version="1.0" encoding="utf-8"?>
 <!DOCTYPE eagle SYSTEM "eagle.dtd">
-<eagle version="6.5.0">
+<eagle version="6.6.0">
 <drawing>
 <settings>
@@
 <wire x1="347.98" y1="185.42" x2="347.98" y2="182.88" width="0.1524" layer="91"/>
 <pinref part="GND1" gate="1" pin="GND"/>
-</segment>
-<segment>
+<pinref part="U6" gate="1" pin="6A"/>
+<wire x1="345.44" y1="190.5" x2="347.98" y2="190.5" width="0.1524" layer="91"/>
+<wire x1="347.98" y1="190.5" x2="347.98" y2="185.42" width="0.1524" layer="91"/>
+<junction x="347.98" y="185.42"/>
+</segment>
+<segment>

Commit message: fixed all issued in github
Parts:
- added FID1, FID2: FIDUCIAL1X2, SparkFun-Aesthetics:FIDUCIAL1X2
- renumbered POWER to D18, PROTECT to D3
Other:
- note added: "Power"
- note added: "Reverse Protect"
Changed lines of the file:
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@@
 <?xml version="1.0" encoding="utf-8"?>
 <!DOCTYPE eagle SYSTEM "eagle.dtd">
-<eagle version="6.6.0">
+<eagle version="6.5.0">
 <drawing>
 <settings>
@@
 <part name="R50" library="SparkFun-Resistors" deviceset="1KOHM1/10W1%(0603)" device="" value="1K"/>
 <part name="GND27" library="SparkFun" deviceset="GND" device=""/>
-<part name="PROTECT" library="SparkFun-LED" deviceset="LED-RED" device="LILYPAD" value="RED"/>
+<part name="D3" library="SparkFun-LED" deviceset="LED-RED" device="LILYPAD" value="RED"/>
 <part name="R51" library="SparkFun-Resistors" deviceset="10KOHM-1/10W-1%(0603)" device="0603" value="10K"/>
 <part name="C2" library="SparkFun-Capacitors" deviceset="0.1UF-100V-10%(0603)" device="" value="0.1uF"/>
@@
 <part name="LOGO1" library="SparkFun-Aesthetics" deviceset="OSHW-LOGO" device="M"/>
 <part name="LOGO2" library="SparkFun-Aesthetics" deviceset="SFE_LOGO_NAME_FLAME" device=".2_INCH" value="SFE_LOGO_NAME_FLAME.2_INCH"/>
-<part name="POWER" library="SparkFun-LED" deviceset="LED-BLUE" device="1206" value="BLUE"/>
+<part name="D18" library="SparkFun-LED" deviceset="LED-BLUE" device="1206" value="BLUE"/>
 <part name="R56" library="SparkFun-Resistors" deviceset="10KOHM-1/10W-1%(0603)" device="0603" value="10K"/>
 <part name="GND66" library="SparkFun" deviceset="GND" device=""/>
@@
 <part name="C45" library="SparkFun-Capacitors" deviceset="0.1UF-25V(+80/-20%)(0603)" device="" value="0.1uF"/>
 <part name="C46" library="SparkFun-Capacitors" deviceset="0.1UF-25V(+80/-20%)(0603)" device="" value="0.1uF"/>
+<part name="FID1" library="SparkFun-Aesthetics" deviceset="FIDUCIAL" device="1X2"/>
+<part name="FID2" library="SparkFun-Aesthetics" deviceset="FIDUCIAL" device="1X2"/>
 </parts>
 <sheets>
@@
 <text x="12.7" y="63.5" size="2.54" layer="94" font="vector" ratio="15" align="bottom-center">-</text>
 <text x="12.7" y="68.58" size="2.54" layer="94" font="vector" ratio="15" align="bottom-center">+</text>
-<wire x1="330.2" y1="35.56" x2="274.32" y2="35.56" width="0.3048" layer="94"/>
-<wire x1="274.32" y1="35.56" x2="274.32" y2="96.52" width="0.3048" layer="94"/>
-<wire x1="274.32" y1="96.52" x2="274.32" y2="121.92" width="0.3048" layer="94"/>
-<wire x1="274.32" y1="121.92" x2="431.8" y2="121.92" width="0.3048" layer="94"/>
+<wire x1="330.2" y1="35.56" x2="274.32" y2="35.56" width="0.3048" layer="97"/>
+<wire x1="274.32" y1="35.56" x2="274.32" y2="96.52" width="0.3048" layer="97"/>
+<wire x1="274.32" y1="96.52" x2="274.32" y2="121.92" width="0.3048" layer="97"/>
+<wire x1="274.32" y1="121.92" x2="431.8" y2="121.92" width="0.3048" layer="97"/>
 <text x="279.4" y="114.3" size="3.81" layer="94">Status LED's</text>
-<wire x1="274.32" y1="96.52" x2="129.54" y2="96.52" width="0.3048" layer="94"/>
+<wire x1="274.32" y1="96.52" x2="129.54" y2="96.52" width="0.3048" layer="97"/>
 <text x="5.08" y="88.9" size="3.81" layer="94">Power Management</text>
-<wire x1="129.54" y1="96.52" x2="0" y2="96.52" width="0.3048" layer="94"/>
-<wire x1="0" y1="180.34" x2="129.54" y2="180.34" width="0.3048" layer="94"/>
-<wire x1="129.54" y1="180.34" x2="129.54" y2="96.52" width="0.3048" layer="94"/>
+<wire x1="129.54" y1="96.52" x2="0" y2="96.52" width="0.3048" layer="97"/>
+<wire x1="0" y1="180.34" x2="129.54" y2="180.34" width="0.3048" layer="97"/>
+<wire x1="129.54" y1="180.34" x2="129.54" y2="96.52" width="0.3048" layer="97"/>
 <text x="5.08" y="172.72" size="3.81" layer="94">Expansion Headers</text>
-<wire x1="129.54" y1="180.34" x2="129.54" y2="279.4" width="0.3048" layer="94"/>
+<wire x1="129.54" y1="180.34" x2="129.54" y2="279.4" width="0.3048" layer="97"/>
 <text x="5.08" y="271.78" size="3.81" layer="94">USB-&gt;Serial</text>
 <text x="134.62" y="271.78" size="3.81" layer="94">Control Logic</text>
+<text x="40.64" y="45.72" size="1.778" layer="97" rot="R270">Reverse Protect</text>
+<text x="81.28" y="38.1" size="1.778" layer="97" rot="R90">Power</text>
 </plain>
 <instances>
@@
 <instance part="R50" gate="G$1" x="53.34" y="55.88" rot="MR270"/>
 <instance part="GND27" gate="1" x="63.5" y="33.02" rot="MR0"/>
-<instance part="PROTECT" gate="G$1" x="45.72" y="48.26" rot="R180"/>
+<instance part="D3" gate="G$1" x="45.72" y="48.26" rot="R180"/>
 <instance part="R51" gate="G$1" x="45.72" y="60.96" rot="MR270"/>
 <instance part="C2" gate="G$1" x="30.48" y="53.34" rot="MR0"/>
@@
 <instance part="LOGO1" gate="G$1" x="314.96" y="10.16"/>
 <instance part="LOGO2" gate="G$1" x="246.38" y="2.54"/>
-<instance part="POWER" gate="G$1" x="76.2" y="50.8"/>
+<instance part="D18" gate="G$1" x="76.2" y="50.8"/>
 <instance part="R56" gate="G$1" x="76.2" y="60.96" rot="MR270"/>
 <instance part="GND66" gate="1" x="76.2" y="40.64" rot="MR0"/>
@@
 <instance part="SUPPLY16" gate="G$1" x="401.32" y="271.78" rot="MR0"/>
 <instance part="GND67" gate="1" x="424.18" y="259.08" rot="MR0"/>
+<instance part="FID1" gate="G$1" x="426.72" y="25.4"/>
+<instance part="FID2" gate="G$1" x="421.64" y="25.4"/>
 </instances>
 <busses>
@@
 </segment>
 <segment>
-<pinref part="POWER" gate="G$1" pin="C"/>
+<pinref part="D18" gate="G$1" pin="C"/>
 <pinref part="GND66" gate="1" pin="GND"/>
 <wire x1="76.2" y1="43.18" x2="76.2" y2="45.72" width="0.1524" layer="91"/>
@@
 <wire x1="35.56" y1="40.64" x2="45.72" y2="40.64" width="0.1524" layer="91"/>
 <junction x="35.56" y="40.64"/>
-<pinref part="PROTECT" gate="G$1" pin="A"/>
+<pinref part="D3" gate="G$1" pin="A"/>
 <wire x1="45.72" y1="40.64" x2="48.26" y2="40.64" width="0.1524" layer="91"/>
 <wire x1="45.72" y1="45.72" x2="45.72" y2="40.64" width="0.1524" layer="91"/>
@@
 <segment>
 <pinref part="R51" gate="G$1" pin="2"/>
-<pinref part="PROTECT" gate="G$1" pin="C"/>
+<pinref part="D3" gate="G$1" pin="C"/>
 <wire x1="45.72" y1="55.88" x2="45.72" y2="53.34" width="0.1524" layer="91"/>
 </segment>
@@
 <segment>
 <pinref part="R56" gate="G$1" pin="2"/>
-<pinref part="POWER" gate="G$1" pin="A"/>
+<pinref part="D18" gate="G$1" pin="A"/>
 <wire x1="76.2" y1="55.88" x2="76.2" y2="53.34" width="0.1524" layer="91"/>
 </segment>
@@
 <text x="287.02" y="269.24" size="6.4516" layer="94" ratio="15">Z-Axis</text>
 <wire x1="147.32" y1="279.4" x2="149.86" y2="279.4" width="0.1524" layer="94"/>
-<wire x1="149.86" y1="279.4" x2="149.86" y2="0" width="0.4064" layer="94"/>
+<wire x1="149.86" y1="279.4" x2="149.86" y2="0" width="0.4064" layer="97"/>
 <wire x1="284.48" y1="279.4" x2="281.94" y2="279.4" width="0.4064" layer="94"/>
-<wire x1="281.94" y1="279.4" x2="281.94" y2="0" width="0.4064" layer="94"/>
+<wire x1="281.94" y1="279.4" x2="281.94" y2="0" width="0.4064" layer="97"/>
 </plain>
 <instances>

Commit message: changes made from github
Changed lines of the file:
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@@
 <layer number="91" name="Nets" color="2" fill="1" visible="yes" active="yes"/>
 <layer number="92" name="Busses" color="1" fill="1" visible="yes" active="yes"/>
-<layer number="93" name="Pins" color="2" fill="1" visible="no" active="yes"/>
+<layer number="93" name="Pins" color="2" fill="1" visible="yes" active="yes"/>
 <layer number="94" name="Symbols" color="4" fill="1" visible="yes" active="yes"/>
 <layer number="95" name="Names" color="7" fill="1" visible="yes" active="yes"/>
@@
 <layer number="99" name="SpiceOrder" color="7" fill="1" visible="yes" active="yes"/>
 <layer number="100" name="Muster" color="7" fill="1" visible="no" active="no"/>
-<layer number="101" name="Patch_Top" color="12" fill="4" visible="no" active="yes"/>
-<layer number="102" name="Vscore" color="7" fill="1" visible="no" active="yes"/>
-<layer number="103" name="tMap" color="7" fill="1" visible="no" active="yes"/>
-<layer number="104" name="Name" color="16" fill="1" visible="no" active="yes"/>
-<layer number="105" name="tPlate" color="7" fill="1" visible="no" active="yes"/>
-<layer number="106" name="bPlate" color="7" fill="1" visible="no" active="yes"/>
-<layer number="107" name="Crop" color="7" fill="1" visible="no" active="yes"/>
+<layer number="101" name="Patch_Top" color="12" fill="4" visible="yes" active="yes"/>
+<layer number="102" name="Vscore" color="7" fill="1" visible="yes" active="yes"/>
+<layer number="103" name="tMap" color="7" fill="1" visible="yes" active="yes"/>
+<layer number="104" name="Name" color="16" fill="1" visible="yes" active="yes"/>
+<layer number="105" name="tPlate" color="7" fill="1" visible="yes" active="yes"/>
+<layer number="106" name="bPlate" color="7" fill="1" visible="yes" active="yes"/>
+<layer number="107" name="Crop" color="7" fill="1" visible="yes" active="yes"/>
 <layer number="108" name="tplace-old" color="10" fill="1" visible="yes" active="yes"/>
 <layer number="109" name="ref-old" color="11" fill="1" visible="yes" active="yes"/>
-<layer number="110" name="fp0" color="7" fill="1" visible="no" active="yes"/>
+<layer number="110" name="fp0" color="7" fill="1" visible="yes" active="yes"/>
 <layer number="111" name="LPC17xx" color="7" fill="1" visible="yes" active="yes"/>
 <layer number="112" name="tSilk" color="7" fill="1" visible="yes" active="yes"/>
 <layer number="113" name="IDFDebug" color="4" fill="1" visible="yes" active="yes"/>
-<layer number="116" name="Patch_BOT" color="9" fill="4" visible="no" active="yes"/>
-<layer number="121" name="_tsilk" color="7" fill="1" visible="no" active="yes"/>
-<layer number="122" name="_bsilk" color="7" fill="1" visible="no" active="yes"/>
-<layer number="123" name="tTestmark" color="7" fill="1" visible="no" active="yes"/>
-<layer number="124" name="bTestmark" color="7" fill="1" visible="no" active="yes"/>
-<layer number="125" name="_tNames" color="7" fill="1" visible="no" active="yes"/>
+<layer number="116" name="Patch_BOT" color="9" fill="4" visible="yes" active="yes"/>
+<layer number="121" name="_tsilk" color="7" fill="1" visible="yes" active="yes"/>
+<layer number="122" name="_bsilk" color="7" fill="1" visible="yes" active="yes"/>
+<layer number="123" name="tTestmark" color="7" fill="1" visible="yes" active="yes"/>
+<layer number="124" name="bTestmark" color="7" fill="1" visible="yes" active="yes"/>
+<layer number="125" name="_tNames" color="7" fill="1" visible="yes" active="yes"/>
 <layer number="126" name="_bNames" color="7" fill="1" visible="yes" active="yes"/>
 <layer number="127" name="_tValues" color="7" fill="1" visible="yes" active="yes"/>
 <layer number="128" name="_bValues" color="7" fill="1" visible="yes" active="yes"/>
 <layer number="129" name="Mask" color="7" fill="1" visible="yes" active="yes"/>
-<layer number="131" name="tAdjust" color="7" fill="1" visible="no" active="yes"/>
-<layer number="132" name="bAdjust" color="7" fill="1" visible="no" active="yes"/>
-<layer number="144" name="Drill_legend" color="7" fill="1" visible="no" active="yes"/>
-<layer number="150" name="Notes" color="7" fill="1" visible="no" active="yes"/>
-<layer number="151" name="HeatSink" color="7" fill="1" visible="no" active="yes"/>
+<layer number="131" name="tAdjust" color="7" fill="1" visible="yes" active="yes"/>
+<layer number="132" name="bAdjust" color="7" fill="1" visible="yes" active="yes"/>
+<layer number="144" name="Drill_legend" color="7" fill="1" visible="yes" active="yes"/>
+<layer number="150" name="Notes" color="7" fill="1" visible="yes" active="yes"/>
+<layer number="151" name="HeatSink" color="7" fill="1" visible="yes" active="yes"/>
 <layer number="152" name="_bDocu" color="7" fill="1" visible="yes" active="yes"/>
 <layer number="153" name="FabDoc1" color="6" fill="1" visible="no" active="no"/>
@@
 <layer number="155" name="FabDoc3" color="7" fill="15" visible="no" active="no"/>
 <layer number="199" name="Contour" color="7" fill="1" visible="yes" active="yes"/>
-<layer number="200" name="200bmp" color="1" fill="10" visible="no" active="yes"/>
-<layer number="201" name="201bmp" color="2" fill="10" visible="no" active="yes"/>
-<layer number="202" name="202bmp" color="3" fill="10" visible="no" active="yes"/>
-<layer number="203" name="203bmp" color="4" fill="10" visible="no" active="yes"/>
-<layer number="204" name="204bmp" color="5" fill="10" visible="no" active="yes"/>
-<layer number="205" name="205bmp" color="6" fill="10" visible="no" active="yes"/>
-<layer number="206" name="206bmp" color="7" fill="10" visible="no" active="yes"/>
-<layer number="207" name="207bmp" color="8" fill="10" visible="no" active="yes"/>
-<layer number="208" name="208bmp" color="9" fill="10" visible="no" active="yes"/>
-<layer number="209" name="209bmp" color="7" fill="1" visible="no" active="yes"/>
-<layer number="210" name="210bmp" color="7" fill="1" visible="no" active="yes"/>
-<layer number="211" name="211bmp" color="7" fill="1" visible="no" active="yes"/>
-<layer number="212" name="212bmp" color="7" fill="1" visible="no" active="yes"/>
-<layer number="213" name="213bmp" color="7" fill="1" visible="no" active="yes"/>
-<layer number="214" name="214bmp" color="7" fill="1" visible="no" active="yes"/>
-<layer number="215" name="215bmp" color="7" fill="1" visible="no" active="yes"/>
-<layer number="216" name="216bmp" color="7" fill="1" visible="no" active="yes"/>
+<layer number="200" name="200bmp" color="1" fill="10" visible="yes" active="yes"/>
+<layer number="201" name="201bmp" color="2" fill="10" visible="yes" active="yes"/>
+<layer number="202" name="202bmp" color="3" fill="10" visible="yes" active="yes"/>
+<layer number="203" name="203bmp" color="4" fill="10" visible="yes" active="yes"/>
+<layer number="204" name="204bmp" color="5" fill="10" visible="yes" active="yes"/>
+<layer number="205" name="205bmp" color="6" fill="10" visible="yes" active="yes"/>
+<layer number="206" name="206bmp" color="7" fill="10" visible="yes" active="yes"/>
+<layer number="207" name="207bmp" color="8" fill="10" visible="yes" active="yes"/>
+<layer number="208" name="208bmp" color="9" fill="10" visible="yes" active="yes"/>
+<layer number="209" name="209bmp" color="7" fill="1" visible="yes" active="yes"/>
+<layer number="210" name="210bmp" color="7" fill="1" visible="yes" active="yes"/>
+<layer number="211" name="211bmp" color="7" fill="1" visible="yes" active="yes"/>
+<layer number="212" name="212bmp" color="7" fill="1" visible="yes" active="yes"/>
+<layer number="213" name="213bmp" color="7" fill="1" visible="yes" active="yes"/>
+<layer number="214" name="214bmp" color="7" fill="1" visible="yes" active="yes"/>
+<layer number="215" name="215bmp" color="7" fill="1" visible="yes" active="yes"/>
+<layer number="216" name="216bmp" color="7" fill="1" visible="yes" active="yes"/>
 <layer number="217" name="217bmp" color="18" fill="1" visible="no" active="no"/>
 <layer number="218" name="218bmp" color="19" fill="1" visible="no" active="no"/>
@@
 <layer number="250" name="Descript" color="3" fill="1" visible="no" active="no"/>
 <layer number="251" name="SMDround" color="12" fill="11" visible="no" active="no"/>
-<layer number="254" name="cooling" color="7" fill="1" visible="no" active="yes"/>
+<layer number="254" name="cooling" color="7" fill="1" visible="yes" active="yes"/>
 <layer number="255" name="routoute" color="7" fill="1" visible="yes" active="yes"/>
 </layers>

Commit message: making changes for second proto round
Parts:
- removed JP16, JP17: 2X6 FEMALE, SparkFun-Connectors:M06X2PTH_FEMALE
- added C47: 0.1uF, SparkFun-Capacitors:0.1UF-25V(+80/-20%)(0603)
- added JP2: M13X22X13, SparkFun-Connectors:M13X22X13
- added R57, R58: 1K, SparkFun-Resistors:1KOHM1/10W1%(0603)
Connections:
- removed net N$44: U3.Y, U7.B
- removed net N$52: U3.A, U6.5Y
- new net ESTOP-LOGIC: JP2.4, R40.2, U6.5Y, U7.B
- new net N$65: R57.2, U2.RXD
- new net N$98: C47.1, U2.VCCD
- new net STEP_EN_LOGIC: R49.2, U3.A, U7.Y
- net 5V: now also JP2.2; no longer JP16.2, R31.2, R41.2, R44.2, R45.2
- net A0-RESET/ABORT: now also JP2.6; no longer JP16.6
- net A1-FEED_HOLD: now also JP2.8; no longer JP16.8
- net A2-CYCLE_START/RESUME: now also JP2.10; no longer JP16.10
- net A3-COOLANT_ENABLE: now also JP2.12; no longer JP16.12
- net A4: now also JP2.14; no longer JP17.2
- net A5-PROBE: now also JP2.16, R44.2; no longer JP17.4
- net A6: now also JP2.24; no longer JP17.12
- net A7: now also JP2.23; no longer JP17.11
- net AREF: now also JP2.19; no longer JP17.7
- net D10-LIM-Y: now also R41.2
- net D9-LIM-X: now also R31.2
- net ESTOP: no longer JP16.4, R40.2
- net GND: now also C47.2, D10.C, D11.C, D14.C, D6.C, JP2.11, JP2.13, JP2.15, JP2.17, JP2.20, JP2.9, R54.1, U4.CSG; no longer JP16.11, JP16.9, JP17.1, JP17.3, JP17.5, JP17.8
- net MISO-D12-LIMIT-Z: now also R45.2
- net MOSI-D11-SPINDLE_PWM: now also JP2.26
- net N$1: now also R58.2, U2.TXD; no longer R54.1, U4.CSG
- net PROBE: no longer D11.C
- net RESET: now also JP2.18; no longer JP17.6
- net RXI: now also JP2.21, R58.1; no longer JP17.9, U2.TXD
- net SCK-D13-SPINDLE_DIR: now also JP2.25
- net STEP_ENABLE: now also U3.Y; no longer R49.2, U7.Y
- net TXO: now also JP2.22, R57.1; no longer JP17.10, U2.RXD
- net VCC: now also JP2.5, JP2.7; no longer JP16.5, JP16.7
- net VIN: now also JP2.1, JP2.3; no longer JP16.1, JP16.3
- net X_LIM: no longer D6.C
- net Y_LIM: no longer D10.C
- net Z_LIM: no longer D14.C
Other:
- moved on the sheet: C53, D1, D2, R18, R9, U3, U7

Commit message: finished modifications from proto review
Connections:
- net 5V: now also R44.2
- net A5-PROBE: now also D11.C; no longer R44.2
- net GND: no longer D11.C
Changed lines of the file:
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@@
 <part name="GND71" library="SparkFun" deviceset="GND" device=""/>
 <part name="GND72" library="SparkFun" deviceset="GND" device=""/>
-<part name="GND73" library="SparkFun" deviceset="GND" device=""/>
+<part name="SUPPLY19" library="SparkFun-Aesthetics" deviceset="5V" device=""/>
 </parts>
 <sheets>
@@
 <instance part="GND71" gate="1" x="347.98" y="58.42"/>
 <instance part="GND72" gate="1" x="383.54" y="58.42"/>
-<instance part="GND73" gate="1" x="408.94" y="58.42"/>
+<instance part="SUPPLY19" gate="G$1" x="408.94" y="86.36" rot="MR0"/>
 </instances>
 <busses>
@@
 <wire x1="309.88" y1="60.96" x2="309.88" y2="63.5" width="0.1524" layer="91"/>
 </segment>
-<segment>
-<pinref part="D11" gate="G$1" pin="C"/>
-<pinref part="GND73" gate="1" pin="GND"/>
-<wire x1="408.94" y1="60.96" x2="408.94" y2="63.5" width="0.1524" layer="91"/>
-</segment>
 </net>
 <net name="AREF" class="0">
@@
 <segment>
 <pinref part="R57" gate="G$1" pin="1"/>
-<wire x1="88.9" y1="241.3" x2="104.14" y2="241.3" width="0.1524" layer="91"/>
-<label x="104.14" y="241.3" size="1.27" layer="95" xref="yes"/>
+<wire x1="88.9" y1="241.3" x2="101.6" y2="241.3" width="0.1524" layer="91"/>
+<label x="101.6" y="241.3" size="1.27" layer="95" xref="yes"/>
 </segment>
 </net>
@@
 <segment>
 <pinref part="R58" gate="G$1" pin="1"/>
-<wire x1="99.06" y1="243.84" x2="104.14" y2="243.84" width="0.1524" layer="91"/>
-<label x="104.14" y="243.84" size="1.27" layer="95" xref="yes"/>
+<wire x1="99.06" y1="243.84" x2="101.6" y2="243.84" width="0.1524" layer="91"/>
+<label x="101.6" y="243.84" size="1.27" layer="95" xref="yes"/>
 </segment>
 </net>
@@
 <wire x1="414.02" y1="269.24" x2="401.32" y2="269.24" width="0.1524" layer="91"/>
 <junction x="401.32" y="269.24"/>
+</segment>
+<segment>
+<pinref part="R44" gate="G$1" pin="2"/>
+<pinref part="SUPPLY19" gate="G$1" pin="5V"/>
+<wire x1="408.94" y1="86.36" x2="408.94" y2="83.82" width="0.1524" layer="91"/>
 </segment>
 </net>
@@
 </segment>
 <segment>
-<pinref part="R44" gate="G$1" pin="2"/>
-<wire x1="408.94" y1="83.82" x2="408.94" y2="86.36" width="0.1524" layer="91"/>
-<label x="408.94" y="86.36" size="1.27" layer="95" rot="R90" xref="yes"/>
+<pinref part="D11" gate="G$1" pin="C"/>
+<wire x1="408.94" y1="63.5" x2="408.94" y2="60.96" width="0.1524" layer="91"/>
+<label x="408.94" y="60.96" size="1.27" layer="95" rot="R270" xref="yes"/>
 </segment>
 </net>
@@
 </segment>
 <segment>
+<wire x1="68.58" y1="119.38" x2="71.12" y2="119.38" width="0.1524" layer="91"/>
+<wire x1="71.12" y1="119.38" x2="71.12" y2="127" width="0.1524" layer="91"/>
 <wire x1="71.12" y1="127" x2="73.66" y2="127" width="0.1524" layer="91"/>
-<label x="71.12" y="127" size="1.27" layer="95" rot="R180" xref="yes"/>
+<label x="68.58" y="119.38" size="1.27" layer="95" rot="R180" xref="yes"/>
 <pinref part="JP2" gate="G$1" pin="25"/>
 </segment>
@@
 <segment>
 <wire x1="88.9" y1="127" x2="91.44" y2="127" width="0.1524" layer="91"/>
+<wire x1="91.44" y1="127" x2="91.44" y2="119.38" width="0.1524" layer="91"/>
+<wire x1="91.44" y1="119.38" x2="93.98" y2="119.38" width="0.1524" layer="91"/>
 <pinref part="JP2" gate="G$1" pin="26"/>
-<label x="91.44" y="127" size="1.27" layer="95" xref="yes"/>
-</segment>
-</net>
+<label x="93.98" y="119.38" size="1.27" layer="95" xref="yes"/>
+</segment>
+</net>

Commit message: made changes and added logos. Added test points
Parts:
- JP19: value M12PTH -> (none)
- JP2: value M13X22X13 -> (none)
- renumbered LOGO2 to LOGO3
Other:
- note added: "Arduino Map"
- note added: "Casey Kuhns"
- note added: "D0- RX D1- TX D2- STEP X D3- STEP Y D4- STEP Z D5- DIR X D6- DIR Y D7- DIR Z D8- STEP EN D9- LIM X D10- LIM Y D11- SPIN PWM D12- LIM Z D13- SPIN DIR A0- RESET/ABORT A1- FEED HOLD A2- CYCLE START A3- COOLANT EN A4- UNUSED A5- PROBE A6- UNUSED A7- UNUSED"
- note added: "v03"
- moved on the sheet: C50, C51, C52, Q1, R6, S4, U1

Commit message: made changes from issues in repo
Other:
- note added: "VIN 12-30VDC"
Changed lines of the file:
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@@
 <wire x1="157.48" y1="160.02" x2="157.48" y2="96.52" width="0.3048" layer="97"/>
 <wire x1="129.54" y1="160.02" x2="157.48" y2="160.02" width="0.3048" layer="97"/>
+<text x="10.16" y="45.72" size="1.778" layer="97" rot="R90">VIN 12-30VDC</text>
 </plain>
 <instances>
