File: Hardware/SparkFun_Stepoko.sch (EAGLE design)
At the start: 178 parts, among them J1 AVR ISP, Q1 16MHZ, Q2 100A/100V, U1 ATMEGA328, U2 CY7C65213, U3 74LVC1G04, U4 LM25011, U5 DRV8811, U6 74HC7014D, U7 7432SE, U8 DRV8811, U9 DRV8811

Commit message: updated version numbers
Other:
- note added: "v04"
- note removed: "v03"
Changed lines of the file:
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@@
 <text x="81.28" y="38.1" size="1.778" layer="97" rot="R90">Power</text>
 <text x="350.52" y="10.16" size="2.54" layer="94">Casey Kuhns</text>
-<text x="421.64" y="7.62" size="2.54" layer="94">v03</text>
+<text x="421.64" y="7.62" size="2.54" layer="94">v04</text>
 <text x="132.08" y="99.06" size="1.778" layer="97">D0- RX
 D1- TX
@@
 <wire x1="284.48" y1="279.4" x2="281.94" y2="279.4" width="0.4064" layer="94"/>
 <wire x1="287.02" y1="279.4" x2="287.02" y2="0" width="0.4064" layer="97"/>
-<text x="421.64" y="7.62" size="2.54" layer="94">v03</text>
+<text x="421.64" y="7.62" size="2.54" layer="94">v04</text>
 <text x="350.52" y="10.16" size="2.54" layer="94">Casey Kuhns</text>
 </plain>

Commit message: corrected issues in github
Parts:
- D10, D14, D6: value YELLOW -> Yellow
- U10: value (none) -> +12v
Changed lines of the file:
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@@
 <layer number="113" name="IDFDebug" color="4" fill="1" visible="yes" active="yes"/>
 <layer number="116" name="Patch_BOT" color="9" fill="4" visible="yes" active="yes"/>
+<layer number="118" name="Rect_Pads" color="7" fill="1" visible="yes" active="yes"/>
 <layer number="121" name="_tsilk" color="7" fill="1" visible="yes" active="yes"/>
 <layer number="122" name="_bsilk" color="7" fill="1" visible="yes" active="yes"/>
@@
 <part name="D4" library="SparkFun-LED" deviceset="LED-GREEN" device="LILYPAD" value="GREEN"/>
 <part name="D5" library="SparkFun-LED" deviceset="LED-RED" device="LILYPAD" value="RED"/>
-<part name="D6" library="SparkFun-LED" deviceset="LED-YELLOW" device="LILYPAD" value="YELLOW"/>
+<part name="D6" library="SparkFun-LED" deviceset="LED-YELLOW" device="LILYPAD" value="Yellow"/>
 <part name="R31" library="SparkFun-Resistors" deviceset="1KOHM-1/10W-1%(0603)" device="" value="1K"/>
 <part name="R32" library="SparkFun-Resistors" deviceset="1KOHM-1/10W-1%(0603)" device="" value="1K"/>
@@
 <part name="D8" library="SparkFun-LED" deviceset="LED-GREEN" device="LILYPAD" value="GREEN"/>
 <part name="D9" library="SparkFun-LED" deviceset="LED-RED" device="LILYPAD" value="RED"/>
-<part name="D10" library="SparkFun-LED" deviceset="LED-YELLOW" device="LILYPAD" value="YELLOW"/>
+<part name="D10" library="SparkFun-LED" deviceset="LED-YELLOW" device="LILYPAD" value="Yellow"/>
 <part name="R41" library="SparkFun-Resistors" deviceset="1KOHM-1/10W-1%(0603)" device="" value="1K"/>
 <part name="R42" library="SparkFun-Resistors" deviceset="1KOHM-1/10W-1%(0603)" device="" value="1K"/>
@@
 <part name="D12" library="SparkFun-LED" deviceset="LED-GREEN" device="LILYPAD" value="GREEN"/>
 <part name="D13" library="SparkFun-LED" deviceset="LED-RED" device="LILYPAD" value="RED"/>
-<part name="D14" library="SparkFun-LED" deviceset="LED-YELLOW" device="LILYPAD" value="YELLOW"/>
+<part name="D14" library="SparkFun-LED" deviceset="LED-YELLOW" device="LILYPAD" value="Yellow"/>
 <part name="R45" library="SparkFun-Resistors" deviceset="1KOHM-1/10W-1%(0603)" device="" value="1K"/>
 <part name="R46" library="SparkFun-Resistors" deviceset="1KOHM-1/10W-1%(0603)" device="" value="1K"/>
@@
 <part name="C40" library="SparkFun-Capacitors" deviceset="47UF-50V-20%(ELECT)" device="" value="47uF"/>
 <part name="GND59" library="SparkFun" deviceset="GND" device=""/>
-<part name="U10" library="SparkFun-PowerIC" deviceset="V_REG_78XX" device="7812"/>
+<part name="U10" library="SparkFun-PowerIC" deviceset="V_REG_78XX" device="7812" value="+12v"/>
 <part name="GND60" library="SparkFun" deviceset="GND" device=""/>
 <part name="C41" library="SparkFun-Capacitors" deviceset="47UF-50V-20%(ELECT)" device="" value="47uF"/>

Commit message: Corrected Probe functionality and updated silk to better reflect limit switch functionality, moved Arduino table to better fit board layout
Parts:
- U2: value CY7C65213 -> FT232RLSSOP; device SparkFun-DigitalIC:CY7C65213 -> SparkFun-DigitalIC:FT232RLSSOP
Connections:
- net A5-PROBE: no longer D11.C
- net N$98: now also U2.3V3OUT; no longer U2.VCCD
- net PROBE: now also D11.C
Changed lines of the file:
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@@
 <part name="S4" library="SparkFun-Electromechanical" deviceset="SWITCH-MOMENTARY-2" device="SMD" value="Reset"/>
 <part name="Q1" library="SparkFun-FreqCtrl" deviceset="RESONATOR" device="16MHZ" value="16MHZ"/>
-<part name="U2" library="SparkFun-DigitalIC" deviceset="CY7C65213" device=""/>
+<part name="U2" library="SparkFun-DigitalIC" deviceset="FT232RL" device="SSOP"/>
 <part name="JP5" library="SparkFun-Connectors" deviceset="USB" device="PTH" value="USB-B"/>
 <part name="JP6" library="SparkFun-Connectors" deviceset="POWER_JACK" device="PTH_LOCK" value="POWER"/>
@@
 <label x="345.44" y="200.914" size="1.27" layer="97" font="vector" ratio="10"/>
 </segment>
+<segment>
+<pinref part="D11" gate="G$1" pin="C"/>
+<wire x1="408.94" y1="63.5" x2="408.94" y2="60.96" width="0.1524" layer="91"/>
+<label x="408.94" y="60.96" size="1.27" layer="95" rot="R270" xref="yes"/>
+</segment>
 </net>
 <net name="N$57" class="0">
@@
 <pinref part="JP2" gate="G$1" pin="16"/>
 </segment>
-<segment>
-<pinref part="D11" gate="G$1" pin="C"/>
-<wire x1="408.94" y1="63.5" x2="408.94" y2="60.96" width="0.1524" layer="91"/>
-<label x="408.94" y="60.96" size="1.27" layer="95" rot="R270" xref="yes"/>
-</segment>
 </net>
 <net name="D4-STEP-Z" class="0">
@@
 <net name="N$98" class="0">
 <segment>
-<pinref part="U2" gate="G$1" pin="VCCD"/>
+<pinref part="U2" gate="G$1" pin="3V3OUT"/>
 <pinref part="C47" gate="G$1" pin="1"/>
 <wire x1="45.72" y1="233.68" x2="33.02" y2="233.68" width="0.1524" layer="91"/>
